File: kicad/fella.kicad_pcb (KiCad board)
At the start: 2 copper layers, 117 parts, among them J1 Conn_02x06_Odd_Even, J2 DE15_Receptacle_HighDensity_M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, J3 USB_C_Receptacle_USB2.0_14P, J4 DE9_Plug_MountingHoles, J5 DB25_Receptacle_MountingHoles, J6 Conn_02x18_Top_Bottom, Q1 BC547, Q2 BC547, SW2 SW_Omron_B3FS, U1 74HC163, U10 TMS4416, U11 TMS4416, U12 TMS4416, U13 74HC157, U14 74HC157, U15 74HC04, U16 74HC32, U17 74HC174, U18 XC9536PC44, U19 74HC574, U2 NE555P, U20 74HC574, U21 74HC245, U22 74HC02, U23 74HC138, U24 6264, U25 74HC574, U26 2764, U27 74HC166, U28 74HC244, U29 6522, U3 74HC138, U30 6551, U31 6551, U32 MAX232, U33 CH340N, U34 24LC256, U35 74HC244, U36 74HC244, U37 74HC245, U4 W65C02SxP, U5 27128, U6 74HC04, U7 74HC00, U8 CY62256-70PC, U9 TMS4416, X1 ACO-25.175MHz-A, X2 ACO-1.8432MHz-A

Commit message: Bugfixes, start routing
Parts:
- added RN3: 4K7x8, Resistor_THT:R_Array_SIP9, F.Cu at (262.9, -97.8)
- added RN4: 4K7x8, Resistor_THT:R_Array_SIP9, F.Cu at (214.6, -129.6)
- R15, R16, R17: value 330R -> 470R
- moved X2 147.5 mm to (262.9, -120.7), turned to -90 degrees
- moved X1 135.5 mm to (129.5, -135.9), turned to 180 degrees
- moved R4 40.7 mm to (139.7, -78.7), turned to 0 degrees
- moved R3 26.7 mm to (129.5, -72.4)
- moved C14 23.1 mm to (160.0, -78.1), turned to 180 degrees
- moved SW2 10.6 mm to (101.0, -74.5), turned to 180 degrees
- moved C13 9.25 mm to (71.2, -108.0)
- moved U5 2.54 mm to (214.6, -106.7)
- moved U8 2.54 mm to (214.6, -125.7)
- moved C15 2.50 mm to (133.3, -82.5)
- moved C43 2.50 mm to (179.1, -149.9), turned to 90 degrees
- moved C5 1.94 mm to (191.8, -137.2)
- moved C6 1.94 mm to (199.4, -137.2)
- moved C7 1.94 mm to (184.2, -137.2)
- moved U32 1.91 mm to (184.2, -142.2)
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Connections:
- J5 pad 22: Net-(J5-P22) -> GND
- J5 pad 23: Net-(J5-P23) -> GND
- U15 pad 12: unconnected-(U15-Pad12) -> Net-(U13-S)
- U15 pad 13: GND -> Net-(U15-Pad13)
- U15 pad 6: Net-(U13-S) -> Net-(U15-Pad13)
- U15 pad 9: Net-(U13-S) -> Net-(U15-Pad13)
- U19 pad 12: /vga/ROW3 -> unconnected-(U19-Q7-Pad12)
- U19 pad 9: /cpu/D7 -> GND
- U20 pad 13: Net-(U20-Q6) -> unconnected-(U20-Q6-Pad13)
- U20 pad 14: Net-(U20-Q5) -> /vga/ROW8
- U20 pad 15: /vga/ROW8 -> /vga/ROW7
- U20 pad 16: /vga/ROW7 -> /vga/ROW6
- U20 pad 17: /vga/ROW6 -> /vga/ROW5
- U20 pad 18: /vga/ROW5 -> /vga/ROW4
- U20 pad 19: /vga/ROW4 -> /vga/ROW3
- U20 pad 8: /cpu/D6 -> GND
- U20 pad 9: /cpu/D7 -> GND
- U22 pad 1: unconnected-(U22-Pad1) -> Net-(U24-~{OE})
- U22 pad 11: Net-(U24-~{OE}) -> Net-(U19-OE)
- U22 pad 12: Net-(U24-~{OE}) -> Net-(U19-OE)
- U22 pad 2: GND -> Net-(U19-OE)
- U22 pad 3: GND -> /cpu/R/W
- U22 pad 8: Net-(U27-Qh) -> /vga/~{BLANK}
- U22 pad 9: /vga/~{BLANK} -> Net-(U27-Qh)
- U23 pad 6: GND -> VCC
- U24 pad 27: /cpu/R/W -> Net-(U24-~{WR})
- U26 pad 2: Net-(U20-Q6) -> /io/ROMSEL1
- U26 pad 23: Net-(U20-Q5) -> /io/ROMSEL0
- U29 pad 14: Net-(J5-P22) -> /io/ROMSEL0
- U29 pad 15: Net-(J5-P23) -> /io/ROMSEL1
- U37 pad 1: Net-(J6-Pin_31) -> Net-(J6-Pin_32)
- U5 pad 20: /cpu//ROMCS -> GND
- U5 pad 22: GND -> /cpu//ROMCS
- U6 pad 12: unconnected-(U6-Pad12) -> Net-(U24-~{WR})
- U6 pad 13: GND -> Net-(U24-~{OE})
- U7 pad 10: GND -> Net-(U7-Pad10)
- U7 pad 11: unconnected-(U7-Pad11) -> /cpu//ROMCS
- U7 pad 12: GND -> Net-(U7-Pad12)
- U7 pad 13: GND -> /cpu//PH2
- U7 pad 2: /cpu//PH2 -> /cpu/A15
- U7 pad 3: /cpu//ROMCS -> Net-(U7-Pad10)
- U7 pad 8: unconnected-(U7-Pad8) -> Net-(U7-Pad12)
- U7 pad 9: GND -> Net-(U7-Pad10)
Routing:
- net /cpu/D3: track 0.00 -> 448.5 mm, vias 0 -> 7
- net /cpu/A1: track 0.00 -> 444.9 mm, vias 0 -> 8
- net /cpu/A0: track 0.00 -> 429.2 mm, vias 0 -> 6
- net /cpu/D4: track 0.00 -> 409.0 mm, vias 0 -> 9
- net /cpu/D6: track 0.00 -> 401.5 mm, vias 0 -> 8
- net /cpu/A2: track 0.00 -> 397.8 mm, vias 0 -> 7
- net /cpu/A3: track 0.00 -> 397.0 mm, vias 0 -> 7
- net /cpu/D5: track 0.00 -> 395.2 mm, vias 0 -> 8
- net /cpu/D0: track 0.00 -> 394.6 mm, vias 0 -> 6
- net /cpu/D1: track 0.00 -> 393.6 mm, vias 0 -> 7
- net /cpu/D2: track 0.00 -> 392.0 mm, vias 0 -> 10
- net /cpu/D7: track 0.00 -> 375.7 mm, vias 0 -> 8
- net /cpu/R/W: track 0.00 -> 356.9 mm, vias 0 -> 9
- net /cpu//RD: track 0.00 -> 331.8 mm, vias 0 -> 4
- net /cpu//RAMCS: track 0.00 -> 278.8 mm, vias 0 -> 4
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Other:
- copper layers 2 -> 4
