File: expansion/emulator/emuprom.kicad_sch (KiCad schematic)
At the start: 33 parts, among them J2 Conn_02x03_Odd_Even, J3 USB_C_Receptacle_USB2.0_14P, U1 CY62256-70PC, U10 74HC244, U2 74HC244, U3 74HC244, U4 74HC244, U5 74HC32, U6 ATmega8-16P, U7 74HC373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

Commit message: emulator: Add crystal value to the schematic
Parts:
- Y1: value Crystal -> 14.7456M
Changed lines of the file:
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@@
 			)
 		)
-		(property "Value" "Crystal"
+		(property "Value" "14.7456M"
 			(at 261.62 109.22 0)
 			(effects
